Commit message: Added a node to switch between manual drive and auto drive mode and fixed flysky driver

File: src/rover_control/urdf/robot.ros2_control.xacro (robot description, xacro)
@@ -3,5 +3,5 @@
     <ros2_control name="GazeboSystemHWI" type="system">
         <hardware>
-            <plugin>gazebo_ros2_control/GazeboSystem</plugin>
+            <plugin>mock_components/GenericSystem</plugin>
         </hardware>
         <joint name="wheel1_joint">

File: src/rover_control/urdf/robot_core_lr.xacro (robot description, xacro)
@@ -1,151 +1,78 @@
 <?xml version="1.0"?>
-<robot xmlns:xacro="http://www.ros.org/wiki/xacro">
-	<material name="white">
-		<color rgba="1 1 1 1"/>
-	</material>
-	<material name="black">
-		<color rgba="0 0 0 1"/>
-	</material>
-	<!-- BASE LINK -->
-	<link name="base_link">
-	</link>
-	<!-- CHASSIS -->
-	<joint name="chassis_joint" type="fixed">
-		<parent link="base_link"/>
-		<child link="chassis_link"/>
-		<origin xyz="0 0 0"/>
-	</joint>
-	<link name="chassis_link">
-		<visual>
-			<origin xyz="0 0 0.1"/>
-			<geometry>
-				<box size="0.8 0.4 0.05"/>
-			</geometry>
-			<material name="white"/>
-		</visual>
-		<collision>
-			<origin xyz="0 0 0.1"/>
-			<geometry>
-				<box size="0.8 0.4 0.05"/>
-			</geometry>
-		</collision>
-		<xacro:inertial_box mass="0.5" x="0.8" y="0.4" z="0.05">
-        	<origin xyz="0 0 0.1" rpy="0 0 0"/>
+<robot xmlns:xacro="http://www.ros.org/wiki/xacro" name="rover">
+    <!-- INERTIAL MACROS (Added these so the xacro tags work) -->
+    <xacro:macro name="inertial_box" params="mass x y z *origin">
+        <inertial>
+            <xacro:insert_block name="origin"/>
+            <mass value="${mass}"/>
+            <inertia ixx="${(1/12) * mass * (y*y + z*z)}" ixy="0.0" ixz="0.0"
+                     iyy="${(1/12) * mass * (x*x + z*z)}" iyz="0.0"
+                     izz="${(1/12) * mass * (x*x + y*y)}"/>
+        </inertial>
+    </xacro:macro>
+    <xacro:macro name="inertial_cylinder" params="mass length radius *origin">
+        <inertial>
+            <xacro:insert_block name="origin"/>
+            <mass value="${mass}"/>
+            <inertia ixx="${(1/12) * mass * (3*radius*radius + length*length)}" ixy="0.0" ixz="0.0"
+                     iyy="${(1/12) * mass * (3*radius*radius + length*length)}" iyz="0.0"
+                     izz="${(1/2) * mass * (radius*radius)}"/>
+        </inertial>
+    </xacro:macro>
+    <material name="white"><color rgba="1 1 1 1"/></material>
+    <material name="black"><color rgba="0 0 0 1"/></material>
+    <!-- BASE LINK -->
+    <link name="base_link"></link>
+    <!-- CHASSIS -->
+    <joint name="chassis_joint" type="fixed">
+        <parent link="base_link"/>
+        <child link="chassis_link"/>
+        <origin xyz="0 0 0"/>
+    </joint>
+    <link name="chassis_link">
+        <visual>
+            <origin xyz="0 0 0.1"/>
+            <geometry><box size="0.8 0.4 0.05"/></geometry>
+            <material name="white"/>
+        </visual>
+        <collision>
+            <origin xyz="0 0 0.1"/>
+            <geometry><box size="0.8 0.4 0.05"/></geometry>
+        </collision>
+        <xacro:inertial_box mass="0.5" x="0.8" y="0.4" z="0.05">
+            <origin xyz="0 0 0.1" rpy="0 0 0"/>
         </xacro:inertial_box>
-	</link>
-	<gazebo reference="chassis">
-		<material>Gazebo/White</material>
-	</gazebo>
-	<!-- WHEEL1 -->
-	<joint name="wheel1_joint" type="continuous">
-		<parent link="base_link"/>
-		<child link="wheel1_link"/>
-		<origin xyz="0.2 0.25 0" rpy="${-pi/2} 0 0"/>
-		<axis xyz="0 0 1"/>
-		<limit effort="10000" velocity="1000" />
-	    <dynamics damping="1.0" friction="1.0" />
-	</joint>
-	<link name="wheel1_link">
-		<visual>
-			<geometry>
-				<cylinder radius="0.1" length="0.1"/>
-			</geometry>
-			<material name="black"/>
-		</visual>
-		<collision>
-			<geometry>
-				<cylinder radius="0.1" length="0.1"/>
-			</geometry>
-		</collision>
-		<xacro:inertial_cylinder mass="0.1" length="0.1" radius="0.1">
-        	<origin xyz="0 0 0" rpy="0 0 0"/>
-        </xacro:inertial_cylinder>
-	</link>
-	<gazebo reference="wheel1_link">
-		<material>Gazebo/Black</material>
-	</gazebo>
-	<!-- WHEEL2 -->
-	<joint name="wheel2_joint" type="continuous">
-		<parent link="base_link"/>
-		<child link="wheel2_link"/>
-		<origin xyz="0.2 -0.25 0" rpy="${pi/2} 0 0"/>
-		<axis xyz="0 0 -1"/>
-		<limit effort="10000" velocity="1000" />
-	    <dynamics damping="1.0" friction="1.0" />
-	</joint>
-	<link name="wheel2_link">
-		<visual>
-			<geometry>
-				<cylinder radius="0.1" length="0.1"/>
-			</geometry>
-			<material name="black"/>
-		</visual>
-		<collision>
-			<geometry>
-				<cylinder radius="0.1" length="0.1"/>
-			</geometry>
-		</collision>
-		<xacro:inertial_cylinder mass="0.1" length="0.1" radius="0.1">
-        	<origin xyz="0 0 0" rpy="0 0 0"/>
-        </xacro:inertial_cylinder>
-	</link>
-	<gazebo reference="wheel2_link">
-		<material>Gazebo/Black</material>
-	</gazebo>
-	<!-- WHEEL3 -->
-	<joint name="wheel3_joint" type="continuous">
-		<parent link="base_link"/>
-		<child link="wheel3_link"/>
-		<origin xyz="-0.2 0.25 0" rpy="${-pi/2} 0 0"/>
-		<axis xyz="0 0 1"/>
-		<limit effort="10000" velocity="1000" />
-	    <dynamics damping="1.0" friction="1.0" />
-	</joint>
-	<link name="wheel3_link">
-		<visual>
-			<geometry>
-				<cylinder radius="0.1" length="0.1"/>
-			</geometry>
-			<material name="black"/>
-		</visual>
-		<collision>
-			<geometry>
-				<cylinder radius="0.1" length="0.1"/>
-			</geometry>
-		</collision>
-		<xacro:inertial_cylinder mass="0.1" length="0.1" radius="0.1">
-        	<origin xyz="0 0 0" rpy="0 0 0"/>
-        </xacro:inertial_cylinder>
-	</link>
-	<gazebo reference="wheel3_link">
-		<material>Gazebo/Black</material>
-	</gazebo>
-	<!-- WHEEL4 -->
-	<joint name="wheel4_joint" type="continuous">
-		<parent link="base_link"/>
-		<child link="wheel4_link"/>
-		<origin xyz="-0.2 -0.25 0" rpy="${pi/2} 0 0"/>
-		<axis xyz="0 0 -1"/>
-		<limit effort="10000" velocity="1000" />
-	    <dynamics damping="1.0" friction="1.0" />
-	</joint>
-	<link name="wheel4_link">
-		<visual>
-			<geometry>
-				<cylinder radius="0.1" length="0.1"/>
-			</geometry>
-			<material name="black"/>
-		</visual>
-		<collision>
-			<geometry>
-				<cylinder radius="0.1" length="0.1"/>
-			</geometry>
-		</collision>
-		<xacro:inertial_cylinder mass="0.1" length="0.1" radius="0.1">
-        	<origin xyz="0 0 0" rpy="0 0 0"/>
-        </xacro:inertial_cylinder>
-	</link>
-	<gazebo reference="wheel4_link">
-		<material>Gazebo/Black</material>
-	</gazebo>
+    </link>
+    <gazebo reference="chassis_link">
+        <material>Gazebo/White</material>
+    </gazebo>
+    <!-- WHEEL MACRO (To clean up the code) -->
+    <xacro:macro name="wheel" params="prefix x_reflect y_reflect">
+        <joint name="${prefix}_wheel_joint" type="continuous">
+            <parent link="base_link"/>
+            <child link="${prefix}_wheel_link"/>
+            <origin xyz="${x_reflect*0.2} ${y_reflect*0.25} 0" rpy="${-pi/2} 0 0"/>
+            <axis xyz="0 0 1"/>
+        </joint>
+        <link name="${prefix}_wheel_link">
+            <visual>
+                <geometry><cylinder radius="0.1" length="0.1"/></geometry>
+                <material name="black"/>
+            </visual>
+            <collision>
+                <geometry><cylinder radius="0.1" length="0.1"/></geometry>
+            </collision>
+            <xacro:inertial_cylinder mass="0.1" length="0.1" radius="0.1">
+                <origin xyz="0 0 0" rpy="0 0 0"/>
+            </xacro:inertial_cylinder>
+        </link>
+        <gazebo reference="${prefix}_wheel_link">
+            <material>Gazebo/Black</material>
+        </gazebo>
+    </xacro:macro>
+    <!-- SPAWN 4 WHEELS -->
+    <xacro:wheel prefix="front_left"  x_reflect="1"  y_reflect="1" />
+    <xacro:wheel prefix="front_right" x_reflect="1"  y_reflect="-1" />
+    <xacro:wheel prefix="back_left"   x_reflect="-1" y_reflect="1" />
+    <xacro:wheel prefix="back_right"  x_reflect="-1" y_reflect="-1" />
 </robot>
